Commit message: Costmap implemented, not working yet

File: install/sentry_description/share/sentry_description/src/description/sentry_description.urdf (robot description, URDF)
Before this commit: robot sentry, 4 links, 3 joints
Links:
- added link lidar_link, mass 0.047; visual box size=${lidar_length} ${lidar_width} ${lidar_height}
Joints:
- added joint lidar_joint: type fixed, parent gimbal_link, child lidar_link, origin xyz=0 0 ${gimbal_height/2 +  lidar_height/2} rpy=0 0 0

File: src/sentry_description/src/description/sentry_description.urdf (robot description, URDF)
Before this commit: robot sentry, 4 links, 3 joints
Links:
- added link lidar_link, mass 0.047; visual box size=${lidar_length} ${lidar_width} ${lidar_height}
Joints:
- added joint lidar_joint: type fixed, parent gimbal_link, child lidar_link, origin xyz=0 0 ${gimbal_height/2 +  lidar_height/2} rpy=0 0 0
