Commit message: Fixed difference between map and world, tweaked radii to enable path planning

File: src/sentry_description/urdf/sentry_description.urdf (robot description, URDF)
Before this commit: robot sentry_robot, 7 links, 6 joints
Links:
- link back_left_wheel: geometry visual cylinder length=0.04 radius=0.05
- link back_right_wheel: geometry visual cylinder length=0.04 radius=0.05
- link front_left_wheel: geometry visual cylinder length=0.04 radius=0.05
- link front_right_wheel: geometry visual cylinder length=0.04 radius=0.05
Joints:
- joint back_left_wheel_joint: origin xyz=-0.15 0.15 0 rpy=0 0 0 -> xyz=-0.15 0.15 -0.11 rpy=0 0 0
- joint back_right_wheel_joint: origin xyz=-0.15 -0.15 0 rpy=0 0 0 -> xyz=-0.15 -0.15 -0.11 rpy=0 0 0
- joint front_left_wheel_joint: origin xyz=0.15 0.15 0 rpy=0 0 0 -> xyz=0.15 0.15 -0.11 rpy=0 0 0
- joint front_right_wheel_joint: origin xyz=0.15 -0.15 0 rpy=0 0 0 -> xyz=0.15 -0.15 -0.11 rpy=0 0 0

Commit message: sentry urdf done

File: src/sentry_description/urdf/sentry_description.urdf (robot description, URDF)
Before this commit: robot sentry_robot, 7 links, 6 joints
Links:
- added link bottom_support_link; collision box size=${support_width * 2 + 2 * gimbal_radius} ${support_length} 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; visual box size=${support_width * 2 + 2 * gimbal_radius} ${support_length} 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
- added link gimbal_link; collision cylinder length=${gimbal_height} radius=${gimbal_radius}; visual cylinder length=${gimbal_height} radius=${gimbal_radius}
- added link gun_shaft_link; visual cylinder length=0.15 radius=0.02
- added link left_support_link; collision box size=${support_width} ${support_length} ${support_standoff_heigh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; visual box size=${support_width} ${support_length} ${support_standoff_heigh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
- added link right_support_link; collision box size=${support_width} ${support_length} ${support_standoff_heigh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; visual box size=${support_width} ${support_length} ${support_standoff_heigh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
- added link turret_link; collision box size=${2*(support_width + gimbal_radius)} ${turret_length} ${tur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; visual box size=${2*(support_width + gimbal_radius)} ${turret_length} ${tur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
- added link turret_shaft_link; visual cylinder length=${2*(support_width + gimbal_radius)} radius=${turret_shaft_radius}
- link base_link: geometry collision box size=${base_width} ${base_length} ${base_height}; visual box size=${base_width} ${base_length} ${base_height}
Joints:
- added joint bottom_support_joint: type fixed, parent gimbal_link, child bottom_support_link, origin xyz=0 0 ${support_base_height / 2} rpy=0 0 0
- added joint gimbal_joint: type continuous, parent base_link, child gimbal_link, origin xyz=0 0 ${base_height + ground_offset + gimbal_height/2} rpy=0 0 0, axis 0 0 1
- added joint gun_shaft_joint: type fixed, parent turret_link, child gun_shaft_link, origin xyz=${turret_length/2 + 0.025} 0 0 rpy=0 1.5708 0, axis 0 0 1
- added joint left_support_joint: type fixed, parent bottom_support_link, child left_support_link, origin xyz=${1.5 * support_width + gimbal_radius} 0 ${(support_standoff_height - support_base_height)/2} rpy=0 0 0
- added joint right_support_joint: type fixed, parent bottom_support_link, child right_support_link, origin xyz=${-(1.5 * support_width + gimbal_radius)} 0 ${(support_standoff_height - support_base_height)/2} rpy=0 0 0
- added joint turret_joint: type fixed, parent turret_shaft_link, child turret_link, origin xyz=0 -0.02 0 rpy=1.5708 0 1.5708
- added joint turret_shaft_joint: type revolute, parent bottom_support_link, child turret_shaft_link, origin xyz=0 0 ${0.75 * support_standoff_height} rpy=0 1.5708 0, axis 0 0 1, limit lower=-0.784 upper=0.784 effort=5 velocity=3.14
- joint back_left_wheel_joint: axis 0 1 0 -> 0 0 1
- joint back_right_wheel_joint: axis 0 1 0 -> 0 0 1
- joint front_left_wheel_joint: axis 0 1 0 -> 0 0 1
- joint front_right_wheel_joint: axis 0 1 0 -> 0 0 1

Commit message: Camera and lidar working

File: src/sentry_description/urdf/sentry_description.urdf (robot description, URDF)
Before this commit: robot sentry_robot, 14 links, 13 joints
Links:
- added link depth_camera_link, mass 0.05; collision box size=0.05 0.05 0.05; visual box size=0.05 0.05 0.05
Joints:
- added joint depth_camera_joint: type fixed, parent turret_link, child depth_camera_link, origin xyz=0.05 0 ${-1 * (turret_height / 2  + 0.025)} rpy=0 0 0
- joint laser_joint: origin xyz=0 0 0.15 rpy=0 0 0 -> xyz=0 0 ${support_standoff_height / 2 + 0.02} rpy=0 0 0; parent base_link -> left_support_link
