Commit message: fixed xacro urdf

File: src/sentry_description/urdf/sentry_description.urdf.xacro (robot description, xacro)
@@ -51,5 +51,4 @@
   <!-- Base Link -->
   <link name="base_link">
-    <origin xyz="0 0 ${base_height/2 + ground_offset}" rpy="0 0 0"/>
     <visual>
       <origin xyz="0 0 ${base_height/2 + ground_offset}" rpy="0 0 0"/>
@@ -91,5 +90,5 @@
     <parent link="base_link"/>
     <child link="front_left_wheel"/>
-    <origin xyz="${base_width/2 + wheel_width/2} ${base_length/2 + wheel_width/2} ${wheel_radius}" rpy="0 1.5708 0"/>
+    <origin xyz="${base_width/2} ${base_length/2} ${ground_offset}" rpy="0 1.5708 0"/>
     <dynamics damping="0.1" friction="0.1"/>
     <axis xyz="0 0 1"/>
@@ -117,5 +116,5 @@
     <parent link="base_link"/>
     <child link="front_right_wheel"/>
-    <origin xyz="${-1 * base_width/2 - wheel_width/2} ${base_length/2 + wheel_width/2} ${wheel_radius}" rpy="0 1.5708 0"/>
+    <origin xyz="${-1 * base_width/2} ${base_length/2} ${ground_offset}" rpy="0 1.5708 0"/>
     <dynamics damping="0.1" friction="0.1"/>
     <axis xyz="0 0 1"/>
@@ -143,5 +142,5 @@
     <parent link="base_link"/>
     <child link="back_left_wheel"/>
-    <origin xyz="${base_width/2 + wheel_width/2} ${-1*base_length/2 - wheel_width/2} ${wheel_radius}" rpy="0 1.5708 0"/>
+    <origin xyz="${base_width/2} ${-1*base_length/2} ${ground_offset}" rpy="0 1.5708 0"/>
     <dynamics damping="0.1" friction="0.1"/>
     <axis xyz="0 0 1"/>
@@ -169,5 +168,5 @@
     <parent link="base_link"/>
     <child link="back_right_wheel"/>
-    <origin xyz="${-1 * base_width/2 - wheel_width/2} ${-1*base_length/2 - wheel_width/2} ${wheel_radius}" rpy="0 1.5708 0"/>
+    <origin xyz="${-1 * base_width/2} ${-1*base_length/2} ${ground_offset}" rpy="0 1.5708 0"/>
     <dynamics damping="0.1" friction="0.1"/>
     <axis xyz="0 0 1"/>
@@ -280,4 +279,10 @@
       </material>
     </visual>
+    <collision>
+      <origin xyz="0 0 0" rpy="0 0 0"/>
+      <geometry>
+        <cylinder radius="${turret_shaft_radius}" length="${2*(support_width + gimbal_radius)}"/>
+      </geometry>
+    </collision>
     <xacro:cylinder_inertia m="${0.5}" rad="${turret_shaft_radius}" h="${2*(support_width + gimbal_radius)}"/>
   </link>
@@ -324,4 +329,11 @@
       </material>
     </visual>
+    <collision>
+      <origin xyz="0 0 0" rpy="0 0 0"/>
+      <geometry>
+        <cylinder radius="0.02" length="0.15"/>
+      </geometry>
+    </collision>
+    <xacro:cylinder_inertia m="0.2" rad="0.02" h="0.15"/>
   </link>
   <joint name="gun_shaft_joint" type="fixed">
@@ -386,4 +398,7 @@
       <box size="0.05 0.05 0.05"/>
     </geometry>
+    <material name="camera_gray">
+      <color rgba="0.5 0.5 0.5 1"/>
+    </material>
   </visual>
   <collision>

Commit message: laser raytracing adjusted, fixed turret joint

File: src/sentry_description/urdf/sentry_description.urdf.xacro (robot description, xacro)
@@ -287,10 +287,10 @@
     <xacro:cylinder_inertia m="${0.5}" rad="${turret_shaft_radius}" h="${2*(support_width + gimbal_radius)}"/>
   </link>
-  <joint name="turret_shaft_joint" type="revolute">
+  <joint name="turret_shaft_joint" type="fixed"> <!-- fixed for now-->
     <parent link="bottom_support_link"/>
     <child link="turret_shaft_link"/>
     <origin xyz="0 0 ${0.75 * support_standoff_height}" rpy="0 1.5708 0"/>
-    <axis xyz="0 0 1"/>
-      <limit lower="-0.784" upper="0.784" effort="5" velocity="3.14"/> <!--not sure good values here-->
+    <!--<axis xyz="0 0 1"/> -->
+      <!-- <limit lower="-0.784" upper="0.784" effort="5" velocity="3.14"/>  -->
   </joint>
   <!-- Turret box -->
@@ -366,7 +366,7 @@
   </link>
   <joint name="laser_joint" type="fixed">
-    <parent link="left_support_link"/>
+    <parent link="turret_link"/>
     <child link="laser_frame"/>
-    <origin xyz="0 0 ${support_standoff_height / 2 + 0.02}" rpy="0 0 0"/>
+    <origin xyz="0.02 ${gimbal_radius + support_width * 1.5} ${-(turret_height / 2 + 0.02)}" rpy="0 0 0"/>
   </joint>
   <!-- IMU -->
@@ -506,6 +506,6 @@
         </scan>
         <range>
-          <min>0.1</min>
-          <max>10.0</max>
+          <min>0.25</min>
+          <max>5</max>
           <resolution>0.01</resolution>
         </range>

Commit message: Added double lidars, merge, serial for comms, republisher, debugged sim robot

File: src/sentry_description/urdf/sentry_description.urdf.xacro (robot description, xacro)
@@ -190,9 +190,10 @@
       <xacro:cylinder_inertia m="0.5" rad="${gimbal_radius}" h="${gimbal_height}"/>
   </link>
-  <joint name="gimbal_joint" type="continuous">
+<!-- changed to fixed -->
+  <joint name="gimbal_joint" type="fixed">
       <parent link="base_link"/>
       <child link="gimbal_link"/>
       <origin xyz="0 0 ${base_height + ground_offset + gimbal_height/2}" rpy="0 0 0"/>
-      <axis xyz="0 0 1"/>
+      <!-- <axis xyz="0 0 1"/> -->
   </joint>
    <!-- support_base -->
@@ -287,10 +288,10 @@
     <xacro:cylinder_inertia m="${0.5}" rad="${turret_shaft_radius}" h="${2*(support_width + gimbal_radius)}"/>
   </link>
-  <joint name="turret_shaft_joint" type="revolute">
+  <joint name="turret_shaft_joint" type="fixed">
     <parent link="bottom_support_link"/>
     <child link="turret_shaft_link"/>
     <origin xyz="0 0 ${0.75 * support_standoff_height}" rpy="0 1.5708 0"/>
-    <axis xyz="0 0 1"/>
-      <limit lower="-0.784" upper="0.784" effort="5" velocity="3.14"/> <!--not sure good values here-->
+    <!-- <axis xyz="0 0 1"/>
+      <limit lower="-0.784" upper="0.784" effort="5" velocity="3.14"/> not sure good values here -->
   </joint>
   <!-- Turret box -->
@@ -344,5 +345,5 @@
   </joint>
   <!-- LiDAR -->
-  <link name="laser_frame">
+  <link name="laser_frame_left">
     <visual>
       <geometry>
@@ -365,7 +366,33 @@
     </inertial>
   </link>
-  <joint name="laser_joint" type="fixed">
+  <joint name="laser_joint_left" type="fixed">
     <parent link="left_support_link"/>
-    <child link="laser_frame"/>
+    <child link="laser_frame_left"/>
+    <origin xyz="0 0 ${support_standoff_height / 2 + 0.02}" rpy="0 0 3.1415926535"/>
+  </joint>
+  <link name="laser_frame_right">
+    <visual>
+      <geometry>
+        <cylinder radius="0.03" length="0.04"/>
+      </geometry>
+      <material name="purple">
+        <color rgba="1 0 1 1"/>
+      </material>
+    </visual>
+    <collision>
+      <geometry>
+        <cylinder radius="0.03" length="0.04"/>
+      </geometry>
+    </collision>
+    <inertial>
+      <mass value="0.1"/>
+      <origin xyz="0 0 0" rpy="0 0 0"/>
+      <inertia ixx="0.0001" ixy="0.0" ixz="0.0"
+               iyy="0.0001" iyz="0.0" izz="0.0001"/>
+    </inertial>
+  </link>
+  <joint name="laser_joint_right" type="fixed">
+    <parent link="right_support_link"/>
+    <child link="laser_frame_right"/>
     <origin xyz="0 0 ${support_standoff_height / 2 + 0.02}" rpy="0 0 0"/>
   </joint>
@@ -388,7 +415,7 @@
   </link>
   <joint name="imu_joint" type="fixed">
-    <parent link="base_link"/>
+    <parent link="gun_shaft_link"/>
     <child link="imu_link"/>
-    <origin xyz="0 0 0.1" rpy="0 0 0"/>
+    <origin xyz="0 0 0" rpy="0 1.5708 0"/>
   </joint>
   <!-- depth camera-->
@@ -465,4 +492,8 @@
   <gazebo>
     <plugin name="planar_move" filename="libgazebo_ros_planar_move.so">
+      <ros>
+        <remapping>cmd_vel:=cmd_vel</remapping>
+        <remapping>odom:=odom</remapping>
+      </ros>
       <update_rate>50</update_rate>
       <publish_rate>50</publish_rate>
@@ -471,9 +502,4 @@
       <odometry_frame>odom</odometry_frame>
       <robot_base_frame>base_link</robot_base_frame>
-      <cmd_vel_topic>cmd_vel</cmd_vel_topic>
-      <odometry_topic>odom</odometry_topic>
-      <covariance_x>0.0001</covariance_x>
-      <covariance_y>0.0001</covariance_y>
-      <covariance_yaw>0.01</covariance_yaw>
     </plugin>
   </gazebo>
@@ -491,6 +517,6 @@
   </gazebo>
   <!-- LiDAR Plugin -->
-  <gazebo reference="laser_frame">
-    <sensor name="laser" type="ray">
+  <gazebo reference="laser_frame_left">
+    <sensor name="laser_left" type="ray">
       <pose>0 0 0 0 0 0</pose>
       <visualize>true</visualize>
@@ -499,8 +525,8 @@
         <scan>
           <horizontal>
-            <samples>360</samples>
+            <samples>241</samples>
             <resolution>1</resolution>
-            <min_angle>-3.14159</min_angle>
-            <max_angle>3.14159</max_angle>
+            <min_angle>1.0471975512</min_angle>
+            <max_angle>5.2359877560</max_angle>
           </horizontal>
         </scan>
@@ -511,10 +537,39 @@
         </range>
       </ray>
-      <plugin name="laser_controller" filename="libgazebo_ros_ray_sensor.so">
+      <plugin name="laser_controller_left" filename="libgazebo_ros_ray_sensor.so">
         <ros>
-          <remapping>~/out:=scan</remapping>
+          <remapping>~/out:=scan_left</remapping>
         </ros>
         <output_type>sensor_msgs/LaserScan</output_type>
-        <frame_name>laser_frame</frame_name>
+        <frame_name>laser_frame_left</frame_name>
+      </plugin>
+    </sensor>
+  </gazebo>
+  <gazebo reference="laser_frame_right">
+    <sensor name="laser_right" type="ray">
+      <pose>0 0 0 0 0 0</pose>
+      <visualize>true</visualize>
+      <update_rate>10</update_rate>
+      <ray>
+        <scan>
+          <horizontal>
+            <samples>121</samples>
+            <resolution>1</resolution>
+            <min_angle>1.0471975512</min_angle>
+            <max_angle>5.2359877560</max_angle>
+          </horizontal>
+        </scan>
+        <range>
+          <min>0.1</min>
+          <max>10.0</max>
+          <resolution>0.01</resolution>
+        </range>
+      </ray>
+      <plugin name="laser_controller_right" filename="libgazebo_ros_ray_sensor.so">
+        <ros>
+          <remapping>~/out:=scan_right</remapping>
+        </ros>
+        <output_type>sensor_msgs/LaserScan</output_type>
+        <frame_name>laser_frame_right</frame_name>
       </plugin>
     </sensor>

Commit message: bug fixes, pathing in progress

File: src/sentry_description/urdf/sentry_description.urdf.xacro (robot description, xacro)
@@ -90,5 +90,5 @@
     <parent link="base_link"/>
     <child link="front_left_wheel"/>
-    <origin xyz="${base_width/2} ${base_length/2} ${ground_offset}" rpy="0 1.5708 0"/>
+    <origin xyz="${base_width/2 - wheel_width/2} ${base_length/2 - wheel_radius} ${ground_offset}" rpy="0 1.5708 0"/>
     <dynamics damping="0.1" friction="0.1"/>
     <axis xyz="0 0 1"/>
@@ -116,5 +116,5 @@
     <parent link="base_link"/>
     <child link="front_right_wheel"/>
-    <origin xyz="${-1 * base_width/2} ${base_length/2} ${ground_offset}" rpy="0 1.5708 0"/>
+    <origin xyz="${-1 * base_width/2 + wheel_width / 2} ${base_length/2 - wheel_radius} ${ground_offset}" rpy="0 1.5708 0"/>
     <dynamics damping="0.1" friction="0.1"/>
     <axis xyz="0 0 1"/>
@@ -142,5 +142,5 @@
     <parent link="base_link"/>
     <child link="back_left_wheel"/>
-    <origin xyz="${base_width/2} ${-1*base_length/2} ${ground_offset}" rpy="0 1.5708 0"/>
+    <origin xyz="${base_width/2 - wheel_width / 2} ${-1*base_length/2 + wheel_radius} ${ground_offset}" rpy="0 1.5708 0"/>
     <dynamics damping="0.1" friction="0.1"/>
     <axis xyz="0 0 1"/>
@@ -168,5 +168,5 @@
     <parent link="base_link"/>
     <child link="back_right_wheel"/>
-    <origin xyz="${-1 * base_width/2} ${-1*base_length/2} ${ground_offset}" rpy="0 1.5708 0"/>
+    <origin xyz="${-1 * base_width/2 + wheel_width / 2} ${-1*base_length/2 + wheel_radius} ${ground_offset}" rpy="0 1.5708 0"/>
     <dynamics damping="0.1" friction="0.1"/>
     <axis xyz="0 0 1"/>
@@ -222,4 +222,28 @@
   </joint>
   <!-- LSL -->
+  <link name="right_support_link">
+    <visual>
+      <origin xyz="0 0 0" rpy="0 0 0"/>
+      <geometry>
+        <box size="${support_width} ${support_length} ${support_standoff_height}"/>
+      </geometry>
+      <material name="red">
+        <color rgba="1 0 0 1"/>
+      </material>
+    </visual>
+    <collision>
+      <origin xyz="0 0 0" rpy="0 0 0"/>
+      <geometry>
+        <box size="${support_width} ${support_length} ${support_standoff_height}"/>
+      </geometry>
+    </collision>
+    <xacro:box_inertia m="${0.5}" w="${support_width}" d="${support_length}" h="${support_standoff_height}"/>
+  </link>
+   <joint name="right_support_joint" type="fixed">
+      <parent link="bottom_support_link"/>
+      <child link="right_support_link"/>
+      <origin xyz="${1.5 * support_width + gimbal_radius} 0 ${(support_standoff_height - support_base_height)/2}" rpy="0 0 0"/>
+  </joint>
+  <!-- RSL -->
   <link name="left_support_link">
     <visual>
@@ -243,28 +267,4 @@
       <parent link="bottom_support_link"/>
       <child link="left_support_link"/>
-      <origin xyz="${1.5 * support_width + gimbal_radius} 0 ${(support_standoff_height - support_base_height)/2}" rpy="0 0 0"/>
-  </joint>
-  <!-- RSL -->
-  <link name="right_support_link">
-    <visual>
-      <origin xyz="0 0 0" rpy="0 0 0"/>
-      <geometry>
-        <box size="${support_width} ${support_length} ${support_standoff_height}"/>
-      </geometry>
-      <material name="red">
-        <color rgba="1 0 0 1"/>
-      </material>
-    </visual>
-    <collision>
-      <origin xyz="0 0 0" rpy="0 0 0"/>
-      <geometry>
-        <box size="${support_width} ${support_length} ${support_standoff_height}"/>
-      </geometry>
-    </collision>
-    <xacro:box_inertia m="${0.5}" w="${support_width}" d="${support_length}" h="${support_standoff_height}"/>
-  </link>
-   <joint name="right_support_joint" type="fixed">
-      <parent link="bottom_support_link"/>
-      <child link="right_support_link"/>
       <origin xyz="${-(1.5 * support_width + gimbal_radius)} 0 ${(support_standoff_height - support_base_height)/2}" rpy="0 0 0"/>
   </joint>
@@ -345,5 +345,5 @@
   </joint>
   <!-- LiDAR -->
-  <link name="laser_frame_left">
+  <link name="laser_frame_right">
     <visual>
       <geometry>
@@ -366,33 +366,33 @@
     </inertial>
   </link>
+  <joint name="laser_joint_right" type="fixed">
+    <parent link="right_support_link"/>
+    <child link="laser_frame_right"/>
+    <origin xyz="0 0 ${support_standoff_height / 2 + 0.02}" rpy="0 0 3.1415926535"/>
+  </joint>
+  <link name="laser_frame_left">
+    <visual>
+      <geometry>
+        <cylinder radius="0.03" length="0.04"/>
+      </geometry>
+      <material name="white">
+        <color rgba="1 1 1 1"/>
+      </material>
+    </visual>
+    <collision>
+      <geometry>
+        <cylinder radius="0.03" length="0.04"/>
+      </geometry>
+    </collision>
+    <inertial>
+      <mass value="0.1"/>
+      <origin xyz="0 0 0" rpy="0 0 0"/>
+      <inertia ixx="0.0001" ixy="0.0" ixz="0.0"
+               iyy="0.0001" iyz="0.0" izz="0.0001"/>
+    </inertial>
+  </link>
   <joint name="laser_joint_left" type="fixed">
     <parent link="left_support_link"/>
     <child link="laser_frame_left"/>
-    <origin xyz="0 0 ${support_standoff_height / 2 + 0.02}" rpy="0 0 3.1415926535"/>
-  </joint>
-  <link name="laser_frame_right">
-    <visual>
-      <geometry>
-        <cylinder radius="0.03" length="0.04"/>
-      </geometry>
-      <material name="purple">
-        <color rgba="1 0 1 1"/>
-      </material>
-    </visual>
-    <collision>
-      <geometry>
-        <cylinder radius="0.03" length="0.04"/>
-      </geometry>
-    </collision>
-    <inertial>
-      <mass value="0.1"/>
-      <origin xyz="0 0 0" rpy="0 0 0"/>
-      <inertia ixx="0.0001" ixy="0.0" ixz="0.0"
-               iyy="0.0001" iyz="0.0" izz="0.0001"/>
-    </inertial>
-  </link>
-  <joint name="laser_joint_right" type="fixed">
-    <parent link="right_support_link"/>
-    <child link="laser_frame_right"/>
     <origin xyz="0 0 ${support_standoff_height / 2 + 0.02}" rpy="0 0 0"/>
   </joint>
@@ -499,5 +499,5 @@
       <publish_rate>50</publish_rate>
       <publish_odom>true</publish_odom>
-      <publish_odom_tf>true</publish_odom_tf>
+      <publish_odom_tf>false</publish_odom_tf>
       <odometry_frame>odom</odometry_frame>
       <robot_base_frame>base_link</robot_base_frame>
@@ -539,5 +539,5 @@
       <plugin name="laser_controller_left" filename="libgazebo_ros_ray_sensor.so">
         <ros>
-          <remapping>~/out:=scan_left</remapping>
+          <remapping>~/out:=/scan_left</remapping>
         </ros>
         <output_type>sensor_msgs/LaserScan</output_type>
@@ -568,5 +568,5 @@
       <plugin name="laser_controller_right" filename="libgazebo_ros_ray_sensor.so">
         <ros>
-          <remapping>~/out:=scan_right</remapping>
+          <remapping>~/out:=/scan_right</remapping>
         </ros>
         <output_type>sensor_msgs/LaserScan</output_type>

Commit message: moved imu to back of turret link

File: src/sentry_description/urdf/sentry_description.urdf.xacro (robot description, xacro)
@@ -415,7 +415,7 @@
   </link>
   <joint name="imu_joint" type="fixed">
-    <parent link="gun_shaft_link"/>
+    <parent link="turret_link"/>
     <child link="imu_link"/>
-    <origin xyz="0 0 0" rpy="0 1.5708 0"/>
+    <origin xyz="${-(support_width + gimbal_radius) + 0.01} ${-turret_length/2 + 0.01} ${-turret_height/2 + 0.005}" rpy="0 0 0"/>
   </joint>
   <!-- depth camera-->

File: src/sentry_description/urdf/sentry_description_v2.urdf.xacro (robot description, xacro)
@@ -448,7 +448,7 @@
   </link>
   <joint name="imu_joint" type="fixed">
-    <parent link="gun_shaft_link"/>
+    <parent link="turret_link"/>
     <child link="imu_link"/>
-    <origin xyz="0 0 0" rpy="0 1.5708 0"/>
+    <origin xyz="${-turret_arm_width/2 + 0.01} ${-turret_length/2 + 0.01} ${-turret_height/2 + 0.005}" rpy="0 0 0"/>
   </joint>
   <!-- ==================== Depth camera ==================== -->

Commit message: updated robot, added ekf with imu position and real robot topics, fixed slam and map function, added keepout, increased wall height

File: src/sentry_description/urdf/sentry_description.urdf.xacro (robot description, xacro)
@@ -190,10 +190,12 @@
       <xacro:cylinder_inertia m="0.5" rad="${gimbal_radius}" h="${gimbal_height}"/>
   </link>
-<!-- changed to fixed -->
-  <joint name="gimbal_joint" type="fixed">
+  <!-- Locked revolute for now: published in /joint_states, but held at 0 rad -->
+  <joint name="gimbal_joint" type="revolute">
       <parent link="base_link"/>
       <child link="gimbal_link"/>
       <origin xyz="0 0 ${base_height + ground_offset + gimbal_height/2}" rpy="0 0 0"/>
-      <!-- <axis xyz="0 0 1"/> -->
+      <axis xyz="0 1 0"/>
+      <limit lower="-0.0001" upper="0.0001" effort="100.0" velocity="0.01"/>
+      <dynamics damping="500.0" friction="100.0"/>
   </joint>
    <!-- support_base -->
@@ -288,10 +290,12 @@
     <xacro:cylinder_inertia m="${0.5}" rad="${turret_shaft_radius}" h="${2*(support_width + gimbal_radius)}"/>
   </link>
-  <joint name="turret_shaft_joint" type="fixed">
+  <!-- Locked revolute for now: published in /joint_states, but held at 0 rad -->
+  <joint name="turret_shaft_joint" type="revolute">
     <parent link="bottom_support_link"/>
     <child link="turret_shaft_link"/>
     <origin xyz="0 0 ${0.75 * support_standoff_height}" rpy="0 1.5708 0"/>
-    <!-- <axis xyz="0 0 1"/>
-      <limit lower="-0.784" upper="0.784" effort="5" velocity="3.14"/> not sure good values here -->
+    <axis xyz="0 0 1"/>
+    <limit lower="-0.0001" upper="0.0001" effort="100.0" velocity="0.01"/>
+    <dynamics damping="500.0" friction="100.0"/>
   </joint>
   <!-- Turret box -->
@@ -499,5 +503,5 @@
       <publish_rate>50</publish_rate>
       <publish_odom>true</publish_odom>
-      <publish_odom_tf>false</publish_odom_tf>
+      <publish_odom_tf>true</publish_odom_tf>
       <odometry_frame>odom</odometry_frame>
       <robot_base_frame>base_link</robot_base_frame>

File: src/sentry_description/urdf/sentry_description_v2.urdf.xacro (robot description, xacro)
@@ -530,5 +530,5 @@
       <publish_rate>50</publish_rate>
       <publish_odom>true</publish_odom>
-      <publish_odom_tf>true</publish_odom_tf>
+      <publish_odom_tf>false</publish_odom_tf>
       <odometry_frame>odom</odometry_frame>
       <robot_base_frame>base_link</robot_base_frame>
