Commit message: URDF WORKING DIMENSIONS, need to move imu

File: src/sentry_description/urdf/sentry_description.urdf.xacro (robot description, xacro)
@@ -2,23 +2,29 @@
 <robot name="sentry_robot" xmlns:xacro="http://ros.org/wiki/xacro">
     <!-- Define robot constants (that we arent using)-->
-  <xacro:property name="base_width" value="0.495"/>
-  <xacro:property name="base_length" value="0.495"/>
-  <xacro:property name="base_height" value="0.15"/>
-  <xacro:property name="ground_offset" value="0.05"/>
-  <xacro:property name="wheel_radius" value="0.1"/>
-  <xacro:property name="wheel_width" value="0.05"/>
+  <xacro:property name="base_width" value="0.540"/>
+  <xacro:property name="base_length" value="0.530"/> <!--in direction of turret-->
+  <xacro:property name="base_height" value="0.066"/>
+  <xacro:property name="ground_offset" value="0.093"/>
+  <xacro:property name="wheel_radius" value="0.075"/>
+  <xacro:property name="wheel_width" value="0.04"/>
   <xacro:property name="wheel_mass" value="0.5"/>
-  <xacro:property name="gimbal_radius" value="0.05"/>
-  <xacro:property name="gimbal_height" value="0.1"/>
+  <xacro:property name="wheel_turret_dir_offset" value="0.2048"/>
+  <xacro:property name="wheel_anti_turret_dir_offset" value="0.1986"/>
+  <xacro:property name="gimbal_radius" value="0.0335"/>
+  <xacro:property name="gimbal_height" value="0.076"/>
   <xacro:property name="lidar_length" value="0.054"/>
   <xacro:property name="lidar_width" value="0.04629"/>
   <xacro:property name="lidar_height" value="0.0348"/>
-  <xacro:property name="support_width" value="0.05"/>
-  <xacro:property name="support_length" value="0.1"/>
+  <xacro:property name="support_width" value="0.3048"/>
+  <xacro:property name="support_length" value="0.0699"/>
   <xacro:property name="support_base_height" value="0.075"/>
-  <xacro:property name="support_standoff_height" value="0.25"/>
+  <xacro:property name="support_standoff_width" value="0.058"/>
+  <xacro:property name="support_standoff_length" value="0.0762"/>
+  <xacro:property name="support_standoff_height" value="0.197"/>
   <xacro:property name="turret_shaft_radius" value="0.01"/>
-  <xacro:property name="turret_length" value="0.15"/>
-  <xacro:property name="turret_height" value="0.075"/>
+  <xacro:property name="turret_length" value="0.18"/>
+  <xacro:property name="turret_width" value="0.262"/>
+  <xacro:property name="turret_height" value="0.15"/>
+  <xacro:property name="turret_height_offset" value="0.03"/>
   <xacro:property name="mass" value="20"/>
   <!-- Define inertial property macros  -->
@@ -90,5 +96,5 @@
     <parent link="base_link"/>
     <child link="front_left_wheel"/>
-    <origin xyz="${base_width/2 - wheel_width/2} ${base_length/2 - wheel_radius} ${ground_offset}" rpy="0 1.5708 0"/>
+    <origin xyz="${wheel_anti_turret_dir_offset} ${wheel_turret_dir_offset} ${wheel_radius}" rpy="0 1.5708 0"/>
     <dynamics damping="0.1" friction="0.1"/>
     <axis xyz="0 0 1"/>
@@ -116,5 +122,5 @@
     <parent link="base_link"/>
     <child link="front_right_wheel"/>
-    <origin xyz="${-1 * base_width/2 + wheel_width / 2} ${base_length/2 - wheel_radius} ${ground_offset}" rpy="0 1.5708 0"/>
+    <origin xyz="${-wheel_anti_turret_dir_offset} ${wheel_turret_dir_offset} ${wheel_radius}" rpy="0 1.5708 0"/>
     <dynamics damping="0.1" friction="0.1"/>
     <axis xyz="0 0 1"/>
@@ -142,5 +148,5 @@
     <parent link="base_link"/>
     <child link="back_left_wheel"/>
-    <origin xyz="${base_width/2 - wheel_width / 2} ${-1*base_length/2 + wheel_radius} ${ground_offset}" rpy="0 1.5708 0"/>
+    <origin xyz="${wheel_anti_turret_dir_offset} ${-wheel_turret_dir_offset} ${wheel_radius}" rpy="0 1.5708 0"/>
     <dynamics damping="0.1" friction="0.1"/>
     <axis xyz="0 0 1"/>
@@ -168,5 +174,5 @@
     <parent link="base_link"/>
     <child link="back_right_wheel"/>
-    <origin xyz="${-1 * base_width/2 + wheel_width / 2} ${-1*base_length/2 + wheel_radius} ${ground_offset}" rpy="0 1.5708 0"/>
+    <origin xyz="${-wheel_anti_turret_dir_offset} ${-wheel_turret_dir_offset} ${wheel_radius}" rpy="0 1.5708 0"/>
     <dynamics damping="0.1" friction="0.1"/>
     <axis xyz="0 0 1"/>
@@ -202,5 +208,5 @@
       <origin xyz="0 0 0" rpy="0 0 0"/>
       <geometry>
-        <box size="${support_width * 2 + 2 * gimbal_radius} ${support_length} ${support_base_height}"/>
+        <box size="${support_width} ${support_length} ${support_base_height}"/>
       </geometry>
       <material name="red">
@@ -211,5 +217,5 @@
       <origin xyz="0 0 0" rpy="0 0 0"/>
       <geometry>
-        <box size="${support_width * 2 + 2 * gimbal_radius} ${support_length} ${support_base_height}"/>
+        <box size="${support_width} ${support_length} ${support_base_height}"/>
       </geometry>
     </collision>
@@ -226,5 +232,5 @@
       <origin xyz="0 0 0" rpy="0 0 0"/>
       <geometry>
-        <box size="${support_width} ${support_length} ${support_standoff_height}"/>
+        <box size="${support_standoff_width} ${support_standoff_length} ${support_standoff_height}"/>
       </geometry>
       <material name="red">
@@ -235,13 +241,13 @@
       <origin xyz="0 0 0" rpy="0 0 0"/>
       <geometry>
-        <box size="${support_width} ${support_length} ${support_standoff_height}"/>
-      </geometry>
-    </collision>
-    <xacro:box_inertia m="${0.5}" w="${support_width}" d="${support_length}" h="${support_standoff_height}"/>
+        <box size="${support_standoff_width} ${support_standoff_length} ${support_standoff_height}"/>
+      </geometry>
+    </collision>
+    <xacro:box_inertia m="${0.5}" w="${support_standoff_width}" d="${support_standoff_length}" h="${support_standoff_height}"/>
   </link>
    <joint name="right_support_joint" type="fixed">
       <parent link="bottom_support_link"/>
       <child link="right_support_link"/>
-      <origin xyz="${1.5 * support_width + gimbal_radius} 0 ${(support_standoff_height - support_base_height)/2}" rpy="0 0 0"/>
+      <origin xyz="${(support_width/2 - support_standoff_width/2)} 0 ${(support_standoff_height - support_base_height)/2}" rpy="0 0 0"/>
   </joint>
   <!-- RSL -->
@@ -250,5 +256,5 @@
       <origin xyz="0 0 0" rpy="0 0 0"/>
       <geometry>
-        <box size="${support_width} ${support_length} ${support_standoff_height}"/>
+        <box size="${support_standoff_width} ${support_standoff_length} ${support_standoff_height}"/>
       </geometry>
       <material name="red">
@@ -259,13 +265,13 @@
       <origin xyz="0 0 0" rpy="0 0 0"/>
       <geometry>
-        <box size="${support_width} ${support_length} ${support_standoff_height}"/>
-      </geometry>
-    </collision>
-    <xacro:box_inertia m="${0.5}" w="${support_width}" d="${support_length}" h="${support_standoff_height}"/>
+        <box size="${support_standoff_width} ${support_standoff_length} ${support_standoff_height}"/>
+      </geometry>
+    </collision>
+    <xacro:box_inertia m="${0.5}" w="${support_standoff_width}" d="${support_standoff_length}" h="${support_standoff_height}"/>
   </link>
    <joint name="left_support_joint" type="fixed">
       <parent link="bottom_support_link"/>
       <child link="left_support_link"/>
-      <origin xyz="${-(1.5 * support_width + gimbal_radius)} 0 ${(support_standoff_height - support_base_height)/2}" rpy="0 0 0"/>
+      <origin xyz="${-(support_width/2 - support_standoff_width/2)} 0 ${(support_standoff_height - support_base_height)/2}" rpy="0 0 0"/>
   </joint>
   <!-- Turret shaft -->
@@ -274,5 +280,5 @@
     <origin xyz="0 0 0" rpy="0 0 0"/>
       <geometry>
-        <cylinder radius="${turret_shaft_radius}" length="${2*(support_width + gimbal_radius)}"/>
+        <cylinder radius="${turret_shaft_radius}" length="${2*(support_width/2 - support_standoff_width/2)}"/>
       </geometry>
       <material name="yellow">
@@ -300,5 +306,5 @@
       <origin xyz="0 0 0" rpy="0 0 0"/>
       <geometry>
-        <box size="${2*(support_width + gimbal_radius)} ${turret_length} ${turret_height}"/>
+        <box size="${turret_width} ${turret_length} ${turret_height}"/>
       </geometry>
       <material name="green">
@@ -309,13 +315,13 @@
       <origin xyz="0 0 0" rpy="0 0 0"/>
       <geometry>
-        <box size="${2*(support_width + gimbal_radius)} ${turret_length} ${turret_height}"/>
-      </geometry>
-    </collision>
-    <xacro:box_inertia m="3" w="${2*(support_width + gimbal_radius)}" d="${turret_length}" h="${turret_height}"/>
+        <box size="${turret_width} ${turret_length} ${turret_height}"/>
+      </geometry>
+    </collision>
+    <xacro:box_inertia m="3" w="${turret_width}" d="${turret_length}" h="${turret_height}"/>
   </link>
    <joint name="turret_joint" type="fixed">
       <parent link="turret_shaft_link"/>
       <child link="turret_link"/>
-      <origin xyz="0 -0.02 0" rpy="1.5708 0 1.5708"/>
+      <origin xyz="${-(turret_height_offset)} -0.014 0" rpy="1.5708 0 1.5708"/>
   </joint>
   <!-- gun barrel shaft -->

Commit message: moved imu link, adjusted some sim parameters

File: src/sentry_description/urdf/sentry_description.urdf.xacro (robot description, xacro)
@@ -427,5 +427,5 @@
     <parent link="turret_link"/>
     <child link="imu_link"/>
-    <origin xyz="${-(support_width + gimbal_radius) + 0.01} ${-turret_length/2 + 0.01} ${-turret_height/2 + 0.005}" rpy="0 0 0"/>
+    <origin xyz="${-(turret_width - 0.02)/2} 0 0" rpy="0 0 0"/>
   </joint>
   <!-- depth camera-->

Commit message: save progress. localization working, needs debuggin, initial yaw offset issue

File: src/sentry_description/urdf/sentry_description.urdf.xacro (robot description, xacro)
@@ -200,8 +200,7 @@
       <parent link="base_link"/>
       <child link="gimbal_link"/>
-      <origin xyz="0 0 ${base_height + ground_offset + gimbal_height/2}" rpy="0 0 0"/>
-      <axis xyz="0 1 0"/>
-      <limit lower="-0.0001" upper="0.0001" effort="100.0" velocity="0.01"/>
-      <dynamics damping="500.0" friction="100.0"/>
+      <origin xyz="0 0 ${base_height + ground_offset + gimbal_height/2}" rpy="0 0 -1.5708"/>
+      <axis xyz="0 0 1"/>
+      <dynamics damping="0.1" friction="0.1"/>
   </joint>
    <!-- support_base -->

Commit message: debugging in progress, turret doesnt spin

File: src/sentry_description/urdf/sentry_description.urdf.xacro (robot description, xacro)
@@ -196,6 +196,5 @@
       <xacro:cylinder_inertia m="0.5" rad="${gimbal_radius}" h="${gimbal_height}"/>
   </link>
-  <!-- Locked revolute for now: published in /joint_states, but held at 0 rad -->
-  <joint name="gimbal_joint" type="revolute">
+  <joint name="gimbal_joint" type="continuous">
       <parent link="base_link"/>
       <child link="gimbal_link"/>

Commit message: everything works, but publish rate of mcb data is too slow at 2hz

File: src/sentry_description/urdf/sentry_description.urdf.xacro (robot description, xacro)
@@ -377,5 +377,5 @@
     <parent link="right_support_link"/>
     <child link="laser_frame_right"/>
-    <origin xyz="0 0 ${support_standoff_height / 2 + 0.02}" rpy="0 0 3.1415926535"/>
+    <origin xyz="0 0 ${support_standoff_height / 2 + 0.02}" rpy="0 0 -1.5708"/>
   </joint>
   <link name="laser_frame_left">
@@ -403,5 +403,5 @@
     <parent link="left_support_link"/>
     <child link="laser_frame_left"/>
-    <origin xyz="0 0 ${support_standoff_height / 2 + 0.02}" rpy="0 0 0"/>
+    <origin xyz="0 0 ${support_standoff_height / 2 + 0.02}" rpy="0 0 1.5708"/>
   </joint>
   <!-- IMU -->

Commit message: update turret and localization config

File: src/sentry_description/urdf/sentry_description.urdf.xacro (robot description, xacro)
@@ -199,5 +199,5 @@
       <parent link="base_link"/>
       <child link="gimbal_link"/>
-      <origin xyz="0 0 ${base_height + ground_offset + gimbal_height/2}" rpy="0 0 -1.5708"/>
+      <origin xyz="0 0 ${base_height + ground_offset + gimbal_height/2}" rpy="0 0 1.5708"/>
       <axis xyz="0 0 1"/>
       <dynamics damping="0.1" friction="0.1"/>

Commit message: working through issues. odom works. turret pos integration in the works.

File: src/sentry_description/urdf/sentry_description.urdf.xacro (robot description, xacro)
@@ -199,5 +199,5 @@
       <parent link="base_link"/>
       <child link="gimbal_link"/>
-      <origin xyz="0 0 ${base_height + ground_offset + gimbal_height/2}" rpy="0 0 1.5708"/>
+      <origin xyz="0 0 ${base_height + ground_offset + gimbal_height/2}" rpy="0 0 ${0 + 1.05/2}"/>
       <axis xyz="0 0 1"/>
       <dynamics damping="0.1" friction="0.1"/>
@@ -377,5 +377,5 @@
     <parent link="right_support_link"/>
     <child link="laser_frame_right"/>
-    <origin xyz="0 0 ${support_standoff_height / 2 + 0.02}" rpy="0 0 -1.5708"/>
+    <origin xyz="0 0 ${support_standoff_height / 2 + 0.02}" rpy="0 0 1.5708"/>
   </joint>
   <link name="laser_frame_left">
@@ -403,5 +403,5 @@
     <parent link="left_support_link"/>
     <child link="laser_frame_left"/>
-    <origin xyz="0 0 ${support_standoff_height / 2 + 0.02}" rpy="0 0 1.5708"/>
+    <origin xyz="0 0 ${support_standoff_height / 2 + 0.02}" rpy="0 0 -1.5708"/>
   </joint>
   <!-- IMU -->

Commit message: more lidar smearing debugging

File: src/sentry_description/urdf/sentry_description.urdf.xacro (robot description, xacro)
@@ -199,5 +199,5 @@
       <parent link="base_link"/>
       <child link="gimbal_link"/>
-      <origin xyz="0 0 ${base_height + ground_offset + gimbal_height/2}" rpy="0 0 ${0 + 1.05/2}"/>
+      <origin xyz="0 0 ${base_height + ground_offset + gimbal_height/2}" rpy="0 0 ${1.5708 + 1.05/2}"/>
       <axis xyz="0 0 1"/>
       <dynamics damping="0.1" friction="0.1"/>

Commit message: more debugging, localization better, odom axis flipped

File: src/sentry_description/urdf/sentry_description.urdf.xacro (robot description, xacro)
@@ -199,5 +199,5 @@
       <parent link="base_link"/>
       <child link="gimbal_link"/>
-      <origin xyz="0 0 ${base_height + ground_offset + gimbal_height/2}" rpy="0 0 ${1.5708 + 1.05/2}"/>
+      <origin xyz="0 0 ${base_height + ground_offset + gimbal_height/2}" rpy="0 0 ${0}"/>
       <axis xyz="0 0 1"/>
       <dynamics damping="0.1" friction="0.1"/>
@@ -377,5 +377,5 @@
     <parent link="right_support_link"/>
     <child link="laser_frame_right"/>
-    <origin xyz="0 0 ${support_standoff_height / 2 + 0.02}" rpy="0 0 1.5708"/>
+    <origin xyz="0 0 ${support_standoff_height / 2 + 0.02}" rpy="0 0 -1.5708"/>
   </joint>
   <link name="laser_frame_left">
@@ -403,5 +403,5 @@
     <parent link="left_support_link"/>
     <child link="laser_frame_left"/>
-    <origin xyz="0 0 ${support_standoff_height / 2 + 0.02}" rpy="0 0 -1.5708"/>
+    <origin xyz="0 0 ${support_standoff_height / 2 + 0.02}" rpy="0 0 1.5708"/>
   </joint>
   <!-- IMU -->

Commit message: odom works, lidar scans are smearing

File: src/sentry_description/urdf/sentry_description.urdf.xacro (robot description, xacro)
@@ -55,6 +55,11 @@
   </inertial>
 </xacro:macro>
-  <!-- Base Link -->
+  <!-- Base Link = turret reference frame. The chassis rotates underneath via chassis_joint.
+       No visual here — chassis box lives on chassis_link. -->
   <link name="base_link">
+    <xacro:box_inertia m="1.0" w="0.05" d="0.05" h="0.05"/>
+  </link>
+  <!-- Chassis link: the rotating base that beyblade under the turret -->
+  <link name="chassis_link">
     <visual>
       <origin xyz="0 0 ${base_height/2 + ground_offset}" rpy="0 0 0"/>
@@ -74,4 +79,12 @@
     <xacro:box_inertia m="${mass}" w="${base_width}" d="${base_length}" h="${base_height}"/>
   </link>
+  <!-- chassis_joint: chassis rotates under the turret (base_link).
+       Position = turret_data[0] from the encoder (chassis CCW angle relative to turret). -->
+  <joint name="chassis_joint" type="continuous">
+    <parent link="base_link"/>
+    <child link="chassis_link"/>
+    <origin xyz="0 0 0" rpy="0 0 0"/>
+    <axis xyz="0 0 1"/>
+  </joint>
   <!-- Front Left Wheel -->
   <link name="front_left_wheel">
@@ -94,5 +107,5 @@
   </link>
   <joint name="front_left_wheel_joint" type="continuous">
-    <parent link="base_link"/>
+    <parent link="chassis_link"/>
     <child link="front_left_wheel"/>
     <origin xyz="${wheel_anti_turret_dir_offset} ${wheel_turret_dir_offset} ${wheel_radius}" rpy="0 1.5708 0"/>
@@ -120,5 +133,5 @@
   </link>
   <joint name="front_right_wheel_joint" type="continuous">
-    <parent link="base_link"/>
+    <parent link="chassis_link"/>
     <child link="front_right_wheel"/>
     <origin xyz="${-wheel_anti_turret_dir_offset} ${wheel_turret_dir_offset} ${wheel_radius}" rpy="0 1.5708 0"/>
@@ -146,5 +159,5 @@
   </link>
   <joint name="back_left_wheel_joint" type="continuous">
-    <parent link="base_link"/>
+    <parent link="chassis_link"/>
     <child link="back_left_wheel"/>
     <origin xyz="${wheel_anti_turret_dir_offset} ${-wheel_turret_dir_offset} ${wheel_radius}" rpy="0 1.5708 0"/>
@@ -172,5 +185,5 @@
   </link>
   <joint name="back_right_wheel_joint" type="continuous">
-    <parent link="base_link"/>
+    <parent link="chassis_link"/>
     <child link="back_right_wheel"/>
     <origin xyz="${-wheel_anti_turret_dir_offset} ${-wheel_turret_dir_offset} ${wheel_radius}" rpy="0 1.5708 0"/>
@@ -196,10 +209,10 @@
       <xacro:cylinder_inertia m="0.5" rad="${gimbal_radius}" h="${gimbal_height}"/>
   </link>
-  <joint name="gimbal_joint" type="continuous">
+  <!-- gimbal_joint is now FIXED: base_link IS the turret frame, so the
+       gimbal structure is rigidly attached. chassis_joint handles rotation. -->
+  <joint name="gimbal_joint" type="fixed">
       <parent link="base_link"/>
       <child link="gimbal_link"/>
       <origin xyz="0 0 ${base_height + ground_offset + gimbal_height/2}" rpy="0 0 1.5708"/>
-      <axis xyz="0 0 1"/>
-      <dynamics damping="0.1" friction="0.1"/>
   </joint>
    <!-- support_base -->
@@ -455,6 +468,6 @@
   <origin xyz="0.05 0 ${-1 * (turret_height / 2  + 0.025)}" rpy="0 0 0"/>
   </joint>
-    <!-- Gazebo-specific properties for base_link -->
-    <gazebo reference="base_link">
+    <!-- Gazebo-specific properties for chassis_link -->
+    <gazebo reference="chassis_link">
     <mu1>0.2</mu1>
     <mu2>0.2</mu2>
@@ -509,5 +522,5 @@
       <publish_odom_tf>true</publish_odom_tf>
       <odometry_frame>odom</odometry_frame>
-      <robot_base_frame>base_link</robot_base_frame>
+      <robot_base_frame>chassis_link</robot_base_frame>
     </plugin>
   </gazebo>
@@ -520,5 +533,5 @@
       <joint_name>back_left_wheel_joint</joint_name>
       <joint_name>back_right_wheel_joint</joint_name>
-      <joint_name>gimbal_joint</joint_name>
+      <joint_name>chassis_joint</joint_name>
       <joint_name>turret_shaft_joint</joint_name>
     </plugin>

Commit message: odom almost works

File: src/sentry_description/urdf/sentry_description.urdf.xacro (robot description, xacro)
@@ -55,5 +55,5 @@
   </inertial>
 </xacro:macro>
-  <!-- Base Link -->
+  <!-- Base Link = chassis. Footprint and odometry follow this frame. -->
   <link name="base_link">
     <visual>
@@ -196,8 +196,9 @@
       <xacro:cylinder_inertia m="0.5" rad="${gimbal_radius}" h="${gimbal_height}"/>
   </link>
+  <!-- gimbal_joint: turret rotates relative to chassis (base_link). -->
   <joint name="gimbal_joint" type="continuous">
       <parent link="base_link"/>
       <child link="gimbal_link"/>
-      <origin xyz="0 0 ${base_height + ground_offset + gimbal_height/2}" rpy="0 0 ${0}"/>
+      <origin xyz="0 0 ${base_height + ground_offset + gimbal_height/2}" rpy="0 0 1.5708"/>
       <axis xyz="0 0 1"/>
       <dynamics damping="0.1" friction="0.1"/>

Commit message: more odom debugging

File: src/sentry_description/urdf/sentry_description.urdf.xacro (robot description, xacro)
@@ -196,10 +196,14 @@
       <xacro:cylinder_inertia m="0.5" rad="${gimbal_radius}" h="${gimbal_height}"/>
   </link>
-  <!-- gimbal_joint: turret rotates relative to chassis (base_link). -->
+  <!-- gimbal_joint: turret rotates relative to chassis (base_link).
+       Axis -z so that positive joint value = CW rotation (from above).
+       Combined with publishing -turretYawPos, a CCW chassis spin (which decreases
+       turretYawPos) produces an increasing joint value → CW physical rotation →
+       correct counter-rotation that keeps the turret stationary in world. -->
   <joint name="gimbal_joint" type="continuous">
       <parent link="base_link"/>
       <child link="gimbal_link"/>
       <origin xyz="0 0 ${base_height + ground_offset + gimbal_height/2}" rpy="0 0 1.5708"/>
-      <axis xyz="0 0 1"/>
+      <axis xyz="0 0 -1"/>
       <dynamics damping="0.1" friction="0.1"/>
   </joint>

Commit message: rotational localization done, odom movement causes smearing

File: src/sentry_description/urdf/sentry_description.urdf.xacro (robot description, xacro)
@@ -330,5 +330,5 @@
       <parent link="turret_shaft_link"/>
       <child link="turret_link"/>
-      <origin xyz="${-(turret_height_offset)} -0.014 0" rpy="1.5708 0 1.5708"/>
+      <origin xyz="${(turret_height_offset)} -0.014 0" rpy="1.5708 0 -1.5708"/>
   </joint>
   <!-- gun barrel shaft -->

Commit message: fixed turret misalignment, decreased ekf rate. odom not publishing due to empty /wheel_speeds - not trasmitting from mcb firmware

File: src/sentry_description/urdf/sentry_description.urdf.xacro (robot description, xacro)
@@ -204,5 +204,5 @@
       <parent link="base_link"/>
       <child link="gimbal_link"/>
-      <origin xyz="0 0 ${base_height + ground_offset + gimbal_height/2}" rpy="0 0 1.5708"/>
+      <origin xyz="0 0 ${base_height + ground_offset + gimbal_height/2}" rpy="0 0 ${1.5708 + 1.05/2}"/>
       <axis xyz="0 0 -1"/>
       <dynamics damping="0.1" friction="0.1"/>
