Commit message: odom might work

File: src/sentry_description/urdf/sentry_description.urdf.xacro (robot description, xacro)
@@ -96,5 +96,5 @@
     <parent link="base_link"/>
     <child link="front_left_wheel"/>
-    <origin xyz="${wheel_anti_turret_dir_offset} ${wheel_turret_dir_offset} ${wheel_radius}" rpy="0 1.5708 0"/>
+    <origin xyz="${wheel_anti_turret_dir_offset} ${wheel_turret_dir_offset} ${wheel_radius}" rpy="1.5708 0 0"/>
     <dynamics damping="0.1" friction="0.1"/>
     <axis xyz="0 0 1"/>
@@ -122,5 +122,5 @@
     <parent link="base_link"/>
     <child link="front_right_wheel"/>
-    <origin xyz="${-wheel_anti_turret_dir_offset} ${wheel_turret_dir_offset} ${wheel_radius}" rpy="0 1.5708 0"/>
+    <origin xyz="${-wheel_anti_turret_dir_offset} ${wheel_turret_dir_offset} ${wheel_radius}" rpy="1.5708 0 0"/>
     <dynamics damping="0.1" friction="0.1"/>
     <axis xyz="0 0 1"/>
@@ -148,5 +148,5 @@
     <parent link="base_link"/>
     <child link="back_left_wheel"/>
-    <origin xyz="${wheel_anti_turret_dir_offset} ${-wheel_turret_dir_offset} ${wheel_radius}" rpy="0 1.5708 0"/>
+    <origin xyz="${wheel_anti_turret_dir_offset} ${-wheel_turret_dir_offset} ${wheel_radius}" rpy="1.5708 0 0"/>
     <dynamics damping="0.1" friction="0.1"/>
     <axis xyz="0 0 1"/>
@@ -174,5 +174,5 @@
     <parent link="base_link"/>
     <child link="back_right_wheel"/>
-    <origin xyz="${-wheel_anti_turret_dir_offset} ${-wheel_turret_dir_offset} ${wheel_radius}" rpy="0 1.5708 0"/>
+    <origin xyz="${-wheel_anti_turret_dir_offset} ${-wheel_turret_dir_offset} ${wheel_radius}" rpy="1.5708 0 0"/>
     <dynamics damping="0.1" friction="0.1"/>
     <axis xyz="0 0 1"/>
@@ -204,5 +204,5 @@
       <parent link="base_link"/>
       <child link="gimbal_link"/>
-      <origin xyz="0 0 ${base_height + ground_offset + gimbal_height/2}" rpy="0 0 ${1.5708 + 1.05/2}"/>
+      <origin xyz="0 0 ${base_height + ground_offset + gimbal_height/2}" rpy="0 0 ${1.05/2}"/>
       <axis xyz="0 0 -1"/>
       <dynamics damping="0.1" friction="0.1"/>

Commit message: localization works, drifting base issue

File: src/sentry_description/urdf/sentry_description.urdf.xacro (robot description, xacro)
@@ -204,5 +204,5 @@
       <parent link="base_link"/>
       <child link="gimbal_link"/>
-      <origin xyz="0 0 ${base_height + ground_offset + gimbal_height/2}" rpy="0 0 ${1.05/2}"/>
+      <origin xyz="0 0 ${base_height + ground_offset + gimbal_height/2}" rpy="0 0 ${1.5708}"/>
       <axis xyz="0 0 -1"/>
       <dynamics damping="0.1" friction="0.1"/>

Commit message: Working babelade and odom and turret and gimbal (dab)

File: src/sentry_description/urdf/sentry_description.urdf.xacro (robot description, xacro)
@@ -428,7 +428,7 @@
   </link>
   <joint name="imu_joint" type="fixed">
-    <parent link="turret_link"/>
+    <parent link="gimbal_link"/>
     <child link="imu_link"/>
-    <origin xyz="${-(turret_width - 0.02)/2} 0 0" rpy="0 0 0"/>
+    <origin xyz="0 0 0" rpy="0 0 0"/>
   </joint>
   <!-- depth camera-->
